Commit message: changing size values to avoid sensor collision error

File: p3dx_description/urdf/pioneer3dx.xacro (robot description, xacro)
@@ -40,5 +40,5 @@
         </visual>
         <collision>
-            <origin xyz="-0.045 0 0.145" rpy="0 0 0" />
+            <origin xyz="-0.045 0 0.145" rpy="0.01 0.01 0.01" />
             <geometry>
                 <box size="0.35 0.25 0.14" />
@@ -97,5 +97,5 @@
             <origin xyz="0 0 0" rpy="0 0 0" />
             <geometry>
-                <box size="0 0 0" />
+                <box size="0.01 0.01 0.01" />
             </geometry>
         </collision>
@@ -130,5 +130,5 @@
             <origin xyz="0 0 0" rpy="0 0 0" />
             <geometry>
-                <box size="0 0 0" />
+                <box size="0.01 0.01 0.01" />
             </geometry>
         </collision>
@@ -193,5 +193,5 @@
             <origin rpy="0 0 0" xyz="0 0 0" />
             <geometry>
-                <box size="0 0 0" />
+                <box size="0.01 0.01 0.01" />
             </geometry>
         </collision>

File: p3dx_description/urdf/pioneer3dx_wheel.xacro (robot description, xacro)
@@ -71,5 +71,5 @@
 				<origin xyz="0 0 0" rpy="0 0 0" />
 				<geometry>
-					<box size="0 0 0" />
+					<box size="0.01 0.01 0.01" />
 				</geometry>
 			</collision>
